File: Hardware/py32f030f18p6/KiCAD/py32f030f18p6.kicad_pcb (KiCad board)
At the start: 2 copper layers, 45.7 x 22.9 mm, 29 parts, among them J5 Conn_01x04_Pin, J6 Conn_01x13_Pin, J7 Conn_01x13_Pin, J8 USB_B_Mini, SW0 SW_Push, U1 CH340K, U3 AP2114HA-3.3TRG1, U4 py32f030f18p6, Y1 16Mhz Crystal

Commit message: Updated firmware, changed pad size on diode to make more hand solder friendly
Build board and verified blink led on latest board back from jlpcb, programmed with swd using reset pin, changed pad size for diode as it was tiny.
Parts:
- D1: value TB6612FNG -> CUS10S30; footprint Diode_SMD:D_SOD-323 -> footprints:D_SOD-323-H
Other:
- board text added: "PY32f030f18p6 REVE"
- board text removed: "PY32f030f18p6 REVD"
Changed lines of the file:
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@@
 		(embedded_fonts no)
 	)
-	(footprint "Diode_SMD:D_SOD-323"
+	(footprint "footprints:D_SOD-323-H"
 		(layer "B.Cu")
 		(at 183.88 101.74)
@@
 			(at 0 1.85 180)
 			(layer "B.SilkS")
+			(hide yes)
 			(effects
 				(font
@@
 			)
 		)
-		(property "Value" "TB6612FNG"
+		(property "Value" "CUS10S30"
 			(at 0.1 -1.9 180)
 			(layer "B.Fab")
@@
 			)
 		)
-		(property "Datasheet" "https://www.lcsc.com/datasheet/C88224.pdf"
+		(property "Datasheet" "https://www.lcsc.com/datasheet/C146335.pdf"
 			(at 0 0 180)
 			(unlocked yes)
@@
 			)
 		)
-		(property "LCSC Part#" "C88224"
+		(property "LCSC Part#" "C146335"
 			(at 0 0 0)
 			(unlocked yes)
@@
 		(attr smd)
 		(fp_line
-			(start -1.61 -0.85)
+			(start -1.8 -0.85)
 			(end 1.05 -0.85)
 			(stroke
@@
 		)
 		(fp_line
-			(start -1.61 0.85)
-			(end -1.61 -0.85)
+			(start -1.8 0.85)
+			(end -1.8 -0.85)
 			(stroke
 				(width 0.12)
@@
 		)
 		(fp_line
-			(start -1.61 0.85)
+			(start -1.8 0.85)
 			(end 1.05 0.85)
 			(stroke
@@
 		)
 		(fp_line
-			(start -1.6 -0.95)
-			(end 1.6 -0.95)
+			(start -1.8 -0.95)
+			(end 1.8 -0.95)
 			(stroke
 				(width 0.05)
@@
 		)
 		(fp_line
-			(start -1.6 0.95)
-			(end -1.6 -0.95)
+			(start -1.8 0.95)
+			(end -1.8 -0.95)
 			(stroke
 				(width 0.05)
@@
 		)
 		(fp_line
-			(start -1.6 0.95)
-			(end 1.6 0.95)
+			(start -1.8 0.95)
+			(end 1.8 0.95)
 			(stroke
 				(width 0.05)
@@
 		)
 		(fp_line
-			(start 1.6 0.95)
-			(end 1.6 -0.95)
+			(start 1.8 0.95)
+			(end 1.8 -0.95)
 			(stroke
 				(width 0.05)
@@
 		)
 		(pad "1" smd roundrect
-			(at -1.05 0)
-			(size 0.6 0.45)
+			(at -1.15 0)
+			(size 0.8 1)
 			(layers "B.Cu" "B.Mask" "B.Paste")
 			(roundrect_rratio 0.25)
@@
 		)
 		(pad "2" smd roundrect
-			(at 1.05 0)
-			(size 0.6 0.45)
+			(at 1.15 0)
+			(size 0.8 1)
 			(layers "B.Cu" "B.Mask" "B.Paste")
 			(roundrect_rratio 0.25)
@@
 			(at 0 1.85 180)
 			(layer "B.SilkS")
+			(hide yes)
 			(effects
 				(font
@@
 		)
 	)
-	(gr_text "PY32f030f18p6\nREVD"
+	(gr_text "PY32f030f18p6\nREVE"
 		(at 173.78 99.54 0)
 		(layer "B.SilkS")
