File: Hardware/py32f030f18p6/KiCAD/py32f030f18p6.kicad_sch (KiCad schematic)
At the start: 29 parts, among them J5 Conn_01x04_Pin, J6 Conn_01x13_Pin, J7 Conn_01x13_Pin, J8 USB_B_Mini, SW0 SW_Push, U1 CH340K, U3 AP2114HA-3.3TRG1, U4 py32f030f18p6, Y1 16Mhz Crystal

Commit message: Updated firmware, changed pad size on diode to make more hand solder friendly
Build board and verified blink led on latest board back from jlpcb, programmed with swd using reset pin, changed pad size for diode as it was tiny.
Parts:
- D1: value TB6612FNG -> CUS10S30; footprint Diode_SMD:D_SOD-323 -> footprints:D_SOD-323-H; symbol Diode:1N5819WS -> symbols:CUS10S30; LCSC Part# C88224 -> C146335
Changed lines of the file:
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@@
 	)
 	(symbol
-		(lib_id "Diode:1N5819WS")
+		(lib_id "symbols:CUS10S30")
 		(at 92.71 161.29 180)
 		(unit 1)
@@
 			)
 		)
-		(property "Value" "TB6612FNG"
+		(property "Value" "CUS10S30"
 			(at 93.0275 157.48 0)
 			(effects
@@
 			)
 		)
-		(property "Footprint" "Diode_SMD:D_SOD-323"
+		(property "Footprint" "footprints:D_SOD-323-H"
 			(at 92.71 156.845 0)
 			(effects
@@
 			)
 		)
-		(property "Datasheet" "https://www.lcsc.com/datasheet/C88224.pdf"
+		(property "Datasheet" "https://www.lcsc.com/datasheet/C146335.pdf"
 			(at 92.71 161.29 0)
 			(effects
@@
 			)
 		)
-		(property "LCSC Part#" "C88224"
+		(property "LCSC Part#" "C146335"
 			(at 92.71 161.29 0)
 			(effects
